File: brineomatic/brineomatic.kicad_pcb (KiCad board)
At the start: 4 copper layers, 90 x 63.8 mm, 101 parts, among them J10 3.5MM, J11 3.5MM, J15 5.08MM, J3 THERM, J6 3.5MM, J7 Conn_01x04, J8 SERVOS, J9 3.5MM, Q1 AO3400A, Q2 AO3400A, Q3 AO3400A, Q4 AO3400A, Q5 AO3400A, U1 ESP32-S3-DEVKITC, U3 ADS1115IDGSR, U4 StepStick TMC2209, U5 XL1509-5.0

Commit message: first pass fully routed
Parts:
- moved D8 9.55 mm to (124.0, 60.7)
- moved R18 4.35 mm to (114.8, 51.3)
- moved C9 3.55 mm to (75.3, 79.7)
- moved R2 3.45 mm to (110.0, 65.9), turned to 180 degrees
- moved Q2 3.25 mm to (110.2, 68.9)
- moved C13 2.45 mm to (113.2, 51.2)
- moved C16 2.45 mm to (109.7, 51.2)
- moved D2 1.80 mm to (75.5, 82.3)
- moved C2 1.08 mm to (145.4, 59.1), turned to 0 degrees
- moved C14 1.00 mm to (116.4, 51.3)
- moved H3 0.71 mm to (149.5, 32.5)
- moved H4 0.71 mm to (149.5, 89.0)
- moved C21 0.65 mm to (72.3, 51.8)
- moved H1 0.54 mm to (74.0, 32.5)
- moved R35 0.50 mm to (70.7, 51.8), turned to -90 degrees
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Connections:
- R17 pad 2: +3.3V -> GND
- U1 pad 10: /Piezo/PIEZO -> unconnected-(U1-GPIO17-Pad10)
- U1 pad 20: unconnected-(U1-GPIO14-Pad20) -> /Piezo/PIEZO
- U1 pad 34: /Servos/SERVO1 -> /Servos/SERVO2
- U1 pad 36: /Servos/SERVO2 -> /Servos/SERVO1
- U1 pad 38: /Stepper Driver/DIAG -> /Stepper Driver/EN
- U1 pad 39: /Stepper Driver/EN -> /Stepper Driver/DIAG
- U1 pad 40: /Stepper Driver/DIR -> /Stepper Driver/STEP
- U1 pad 41: /Stepper Driver/STEP -> /Stepper Driver/DIR
Routing:
- net +3.3V: track 0.00 -> 289.5 mm, vias 0 -> 1
- net +24V: track 0.00 -> 262.9 mm
- net +5V: track 0.00 -> 164.4 mm
- net TMC2209_RX: track 0.00 -> 73.9 mm, vias 0 -> 2
- net ESP32_5V: track 0.00 -> 64.3 mm, vias 0 -> 2
- net /Stepper Driver/DIR: track 0.00 -> 57.1 mm, vias 0 -> 1
- net /Stepper Driver/STEP: track 0.00 -> 53.6 mm, vias 0 -> 1
- net /Stepper Driver/RX: track 0.00 -> 47.3 mm, vias 0 -> 1
- net /Piezo/PIEZO: track 0.00 -> 45.5 mm
- net /Solenoid Driver 4/INPUT: track 1.60 -> 46.1 mm
- net /Servos/SERVO2: track 0.00 -> 37.7 mm
- net /Stepper Driver/EN: track 0.00 -> 34.8 mm, vias 0 -> 1
- net /Stepper Driver/DIAG: track 0.00 -> 34.8 mm, vias 0 -> 1
- net /Servos/SERVO1: track 0.00 -> 28.5 mm
- net /Solenoid Driver 3/INPUT: track 1.60 -> 28.7 mm
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Other:
- board size 90 x 63.8 mm -> 90 x 63.5 mm
- board text added: "2 1"
