File: brineomatic/brineomatic.kicad_pcb (KiCad board)
At the start: 4 copper layers, 106 x 67.5 mm, 168 parts, among them J11 3.5MM, J13 3.5MM, J15 3.5MM, J18 USB_TYPE_C_16PIN, J20 Conn_01x04, J6 3.5MM, J9 5.08MM, Q1 AO3400A, Q2 AO3400A, Q3 20N06, Q4 AO3400A, Q5 AO3400A, Q6 AO3400A, Q7 FDC6330L, Q8 S8050, Q9 S8050, SW1 RESET, SW2 BOOT, U1 ADS1115IDGSR, U2 LM74700, U3 XL1509-5.0, U4 ESP32-S3-WROOM-1-N16R8, U5 USBLC6-2SC6, U6 XC6210B332MR, U7 CH334F, U8 CH343P, U9 TMC2209-LA, Y1 12Mhz, Y2 32.768kHz

Commit message: a few last minute routing tweaks
Routing:
- net TMC2209_EN: track 83.7 -> 75.5 mm
- net GND: track 33.8 -> 29.2 mm, vias 105 -> 108
- net +24V: track 309.5 -> 310.1 mm
Other:
- outline, holes or cut-outs redrawn
Changed lines of the file:
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@@
 		(sheetname "/")
 		(sheetfile "brineomatic.kicad_sch")
-		(attr exclude_from_pos_files exclude_from_bom allow_missing_courtyard)
+		(attr exclude_from_pos_files exclude_from_bom)
 		(fp_poly
 			(pts
@@
 		)
 		(group ""
-			(members "78bfbaf9-8112-4f02-b881-75418301f28c" "e159566d-f43a-4c7b-85d3-02dbab586e8d")
+			(members "20b7cd7e-f357-4440-adb9-b103820eedb9" "407439e8-89db-4c32-8ed5-947ee85bd7d3")
 		)
 		(embedded_fonts no)
@@
 	)
 	(gr_line
-		(start 66 83.2)
-		(end 68.75 83.2)
+		(start 66 85.5)
+		(end 68.75 85.5)
 		(stroke
 			(width 0.05)
-			(type default)
+			(type solid)
 		)
 		(layer "Edge.Cuts")
@@
 	)
 	(gr_line
-		(start 68.75 83.2)
-		(end 68.75 36.2)
+		(start 68.75 85.5)
+		(end 68.75 36)
 		(stroke
 			(width 0.05)
@@
 	)
 	(gr_arc
-		(start 63 86.2)
-		(mid 63.87868 84.07868)
-		(end 66 83.2)
+		(start 63 88.5)
+		(mid 63.87868 86.37868)
+		(end 66 85.5)
 		(stroke
 			(width 0.05)
@@
 	)
 	(gr_arc
-		(start 66 36.2)
-		(mid 63.87868 35.32132)
-		(end 63 33.2)
+		(start 66 36)
+		(mid 63.87868 35.12132)
+		(end 63 33)
 		(stroke
 			(width 0.05)
@@
 	)
 	(gr_line
-		(start 63 86.2)
+		(start 63 88.5)
 		(end 63 89.5)
 		(stroke
@@
 	)
 	(gr_line
-		(start 68.75 36.2)
-		(end 66 36.2)
+		(start 68.75 36)
+		(end 66 36)
 		(stroke
 			(width 0.05)
@@
 	(gr_line
 		(start 63 32)
-		(end 63 33.2)
+		(end 63 33)
 		(stroke
 			(width 0.05)
@@
 	(segment
 		(start 150.9875 40.2)
-		(end 150.9875 41.4175)
+		(end 150.9875 41.2)
 		(width 0.5)
 		(layer "F.Cu")
@@
 	)
 	(segment
+		(start 150.9875 41.2)
+		(end 150.9875 41.4175)
+		(width 0.5)
+		(layer "F.Cu")
+		(net 1)
+	)
+	(segment
 		(start 112.86 45.54)
 		(end 111.74 45.54)
@@
 	)
 	(segment
-		(start 159.801 40)
-		(end 159.801 37.751)
-		(width 0.5)
-		(layer "F.Cu")
-		(net 1)
-	)
-	(segment
 		(start 158.37 43.85)
 		(end 156.92 43.85)
@@
 	)
 	(segment
-		(start 152.05 37.6)
-		(end 152.05 40)
-		(width 0.5)
-		(layer "F.Cu")
-		(net 1)
-	)
-	(segment
 		(start 94.4 71.5)
 		(end 93.6 70.7)
@@
 	)
 	(via
+		(at 160.9 38.8)
+		(size 0.45)
+		(drill 0.3)
+		(layers "F.Cu" "B.Cu")
+		(free yes)
+		(net 1)
+	)
+	(via
 		(at 160.95 36.1)
 		(size 0.6)
@@
 	)
 	(via
+		(at 150.9875 41.2)
+		(size 0.45)
+		(drill 0.3)
+		(layers "F.Cu" "B.Cu")
+		(net 1)
+	)
+	(via
 		(at 90.5 79.8)
 		(size 0.6)
@@
 	)
 	(via
+		(at 150.9 38.8)
+		(size 0.45)
+		(drill 0.3)
+		(layers "F.Cu" "B.Cu")
+		(free yes)
+		(net 1)
+	)
+	(via
 		(at 97 81.1)
 		(size 0.6)
@@
 	)
 	(segment
+		(start 152.899 41.499)
+		(end 153.2 41.8)
+		(width 0.5)
+		(layer "F.Cu")
+		(net 4)
+	)
+	(segment
 		(start 147.9925 54.755)
 		(end 140.21 54.755)
@@
 	)
 	(segment
+		(start 152.899 38.601)
+		(end 152.899 41.499)
+		(width 0.5)
+		(layer "F.Cu")
+		(net 4)
+	)
+	(segment
 		(start 148.8 47.1)
 		(end 148.8 45.1)
@@
 	)
 	(segment
-		(start 152.899 38.801)
-		(end 152.899 41.549)
-		(width 0.5)
-		(layer "F.Cu")
-		(net 4)
-	)
-	(segment
 		(start 151.25 60.35)
 		(end 153.2 62.3)
@@
 	)
 	(segment
+		(start 152.899 41.549)
+		(end 153.2 41.85)
+		(width 0.5)
+		(layer "F.Cu")
+		(net 4)
+	)
+	(segment
 		(start 158.876 41.674)
 		(end 158.75 41.8)
@@
 	)
 	(segment
-		(start 152.899 41.549)
-		(end 153.2 41.85)
-		(width 0.5)
-		(layer "F.Cu")
-		(net 4)
-	)
-	(segment
 		(start 145.66 81.9)
 		(end 145.66 87.7)
@@
 	)
 	(via
-		(at 153.2 41.85)
+		(at 153.2 41.8)
 		(size 0.6)
 		(drill 0.3)
@@
 	)
 	(via
-		(at 152.5 41.85)
+		(at 152.5 41.8)
 		(size 0.6)
 		(drill 0.3)
@@
 	)
 	(segment
-		(start 148 44.9)
-		(end 148 50.9)
-		(width 0.2)
+		(start 88.5 61.605)
+		(end 89.645 61.605)
+		(width 0.25)
 		(layer "F.Cu")
 		(net 40)
 	)
 	(segment
-		(start 88.5 61.605)
-		(end 89.645 61.605)
-		(width 0.25)
+		(start 128.9 43.5)
+		(end 130 42.4)
+		(width 0.2)
 		(layer "F.Cu")
 		(net 40)
 	)
 	(segment
-		(start 149.05 43.85)
-		(end 148 44.9)
+		(start 90.293534 61.400019)
+		(end 92.224981 61.400019)
 		(width 0.2)
 		(layer "F.Cu")
@@
 	)
 	(segment
-		(start 148 50.9)
-		(end 149 51.9)
+		(start 130 42.4)
+		(end 147.2 42.4)
 		(width 0.2)
 		(layer "F.Cu")
@@
 	)
 	(segment
-		(start 90.293534 61.400019)
-		(end 92.224981 61.400019)
+		(start 148.65 43.85)
+		(end 153.47 43.85)
 		(width 0.2)
 		(layer "F.Cu")
@@
 	)
 	(segment
-		(start 153.47 43.85)
-		(end 149.05 43.85)
+		(start 147.2 42.4)
+		(end 148.65 43.85)
 		(width 0.2)
 		(layer "F.Cu")
@@
 	)
 	(via
-		(at 90.293534 61.400019)
+		(at 128.9 43.5)
 		(size 0.6)
 		(drill 0.3)
@@
 	)
 	(via
-		(at 149 51.9)
-		(size 0.45)
+		(at 90.293534 61.400019)
+		(size 0.6)
 		(drill 0.3)
 		(layers "F.Cu" "B.Cu")
@@
 	)
 	(segment
-		(start 149 58.6)
-		(end 149 51.9)
-		(width 0.2)
+		(start 90.293534 61.400019)
+		(end 101.699981 61.400019)
+		(width 0.25)
 		(layer "B.Cu")
 		(net 40)
 	)
 	(segment
-		(start 146.199981 61.400019)
-		(end 149 58.6)
-		(width 0.2)
+		(start 119.6 43.5)
+		(end 128.9 43.5)
+		(width 0.25)
 		(layer "B.Cu")
 		(net 40)
 	)
 	(segment
-		(start 90.293534 61.400019)
-		(end 146.199981 61.400019)
-		(width 0.2)
+		(start 101.699981 61.400019)
+		(end 119.6 43.5)
+		(width 0.25)
 		(layer "B.Cu")
 		(net 40)
@@
 		(polygon
 			(pts
-				(xy 154.55 42.8) (xy 153.75 42.8) (xy 153.25 42.3) (xy 151.45 42.3) (xy 151.45 41.4) (xy 153.95 41.4)
+				(xy 154.55 42.8) (xy 153.75 42.8) (xy 153.25 42.3) (xy 151.45 42.3) (xy 151.45 41.3) (xy 153.85 41.3)
 				(xy 154.55 42)
 			)
