File: brineomatic/esp32-s3.kicad_sch (KiCad schematic)
At the start: 47 parts, among them J18 USB_TYPE_C_16PIN, Q7 FDC6330L, Q8 S8050, Q9 S8050, SW1 RESET, SW2 BOOT, U4 ESP32-S3-WROOM-1-N16R8, U5 USBLC6-2SC6, U6 XC6210B332MR, U7 CH334F, U8 CH343P, Y1 12Mhz, Y2 32.768kHz

Commit message: fully routed and erc/drc passed
Parts:
- U4: footprint RF_Module:ESP32-S3-WROOM-1 -> yarrboard:ESP32-S3-WROOM-1
- U7: footprint Package_DFN_QFN:QFN-24-1EP_4x4mm_P0.5mm_EP2.7x2.7mm_ThermalVias -> yarrboard:QFN-24-1EP_4x4mm_P0.5mm_EP2.7x2.7mm_ThermalVias
- U8: footprint Package_DFN_QFN:QFN-16-1EP_3x3mm_P0.5mm_EP1.7x1.7mm_ThermalVias -> yarrboard:QFN-16-1EP_3x3mm_P0.5mm_EP1.7x1.7mm_ThermalVias
Changed lines of the file:
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@@
 	(label "USB_D+"
 		(at 68.58 67.31 180)
-		(fields_autoplaced yes)
 		(effects
 			(font
@@
 			(justify right bottom)
 		)
-		(property "Netclass" "DP_90R"
-			(at 68.58 68.58 0)
-			(effects
-				(font
-					(size 1.27 1.27)
-					(italic yes)
-				)
-				(justify right)
-				(hide yes)
-			)
-		)
 	)
 	(label "USB_D-"
 		(at 68.58 69.85 180)
-		(fields_autoplaced yes)
 		(effects
 			(font
@@
 			(justify right bottom)
 		)
-		(property "Netclass" "DP_90R"
-			(at 68.58 71.12 0)
-			(effects
-				(font
-					(size 1.27 1.27)
-					(italic yes)
-				)
-				(justify right)
-				(hide yes)
-			)
-		)
 	)
 	(label "UART_D-"
 		(at 242.57 50.8 180)
-		(fields_autoplaced yes)
 		(effects
 			(font
@@
 			(justify right bottom)
 		)
-		(property "Netclass" "DP_90R"
-			(at 242.57 52.07 0)
-			(effects
-				(font
-					(size 1.27 1.27)
-					(italic yes)
-				)
-				(justify right)
-				(hide yes)
-			)
-		)
 	)
 	(label "RTS"
@@
 			(justify right bottom)
 		)
-		(property "Netclass" "DP_90R"
-			(at 146.304 49.784 0)
-			(effects
-				(font
-					(size 1.27 1.27)
-					(italic yes)
-				)
-				(justify right)
-				(hide yes)
-			)
-		)
 	)
 	(label "UART_D+"
 		(at 242.57 48.26 180)
-		(fields_autoplaced yes)
 		(effects
 			(font
@@
 			(justify right bottom)
 		)
-		(property "Netclass" "DP_90R"
-			(at 242.57 49.53 0)
-			(effects
-				(font
-					(size 1.27 1.27)
-					(italic yes)
-				)
-				(justify right)
-				(hide yes)
-			)
-		)
 	)
 	(label "DTR"
@@
 	(label "HUB_D+"
 		(at 78.74 67.31 0)
-		(fields_autoplaced yes)
 		(effects
 			(font
@@
 			(justify left bottom)
 		)
-		(property "Netclass" "DP_90R"
-			(at 78.74 68.58 0)
-			(effects
-				(font
-					(size 1.27 1.27)
-					(italic yes)
-				)
-				(justify left)
-				(hide yes)
-			)
-		)
 	)
 	(label "CC2_1"
@@
 	(label "VBUS"
 		(at 44.45 33.02 0)
-		(fields_autoplaced yes)
 		(effects
 			(font
@@
 			(justify left bottom)
 		)
-		(property "Netclass" "VBUS"
-			(at 44.45 34.29 0)
-			(effects
-				(font
-					(size 1.27 1.27)
-					(italic yes)
-				)
-				(justify left)
-			)
-		)
 	)
 	(label "UART_D+"
 		(at 193.04 30.48 0)
-		(fields_autoplaced yes)
 		(effects
 			(font
@@
 			(justify left bottom)
 		)
-		(property "Netclass" "DP_90R"
-			(at 193.04 31.75 0)
-			(effects
-				(font
-					(size 1.27 1.27)
-					(italic yes)
-				)
-				(justify left)
-				(hide yes)
-			)
-		)
 	)
 	(label "HUB_D-"
 		(at 78.74 69.85 0)
-		(fields_autoplaced yes)
 		(effects
 			(font
@@
 			(justify left bottom)
 		)
-		(property "Netclass" "DP_90R"
-			(at 78.74 71.12 0)
-			(effects
-				(font
-					(size 1.27 1.27)
-					(italic yes)
-				)
-				(justify left)
-				(hide yes)
-			)
-		)
 	)
 	(label "RTS"
@@
 			(justify right bottom)
 		)
-		(property "Netclass" "DP_90R"
-			(at 146.304 47.244 0)
-			(effects
-				(font
-					(size 1.27 1.27)
-					(italic yes)
-				)
-				(justify right)
-				(hide yes)
-			)
-		)
 	)
 	(label "USB_D+"
 		(at 45.72 52.07 0)
-		(fields_autoplaced yes)
 		(effects
 			(font
@@
 			(justify left bottom)
 		)
-		(property "Netclass" "DP_90R"
-			(at 45.72 53.34 0)
-			(effects
-				(font
-					(size 1.27 1.27)
-					(italic yes)
-				)
-				(justify left)
-			)
-		)
 	)
 	(label "VBUS"
@@
 	(label "UART_D-"
 		(at 193.04 33.02 0)
-		(fields_autoplaced yes)
 		(effects
 			(font
@@
 			(justify left bottom)
 		)
-		(property "Netclass" "DP_90R"
-			(at 193.04 34.29 0)
-			(effects
-				(font
-					(size 1.27 1.27)
-					(italic yes)
-				)
-				(justify left)
-				(hide yes)
-			)
-		)
 	)
 	(label "DTR"
@@
 	(label "USB_D-"
 		(at 45.72 46.99 0)
-		(fields_autoplaced yes)
 		(effects
 			(font
@@
 			(justify left bottom)
 		)
-		(property "Netclass" "DP_90R"
-			(at 45.72 48.26 0)
-			(effects
-				(font
-					(size 1.27 1.27)
-					(italic yes)
-				)
-				(justify left)
-			)
-		)
 	)
 	(label "VBUS"
@@
 		(shape input)
 		(at 191.77 43.18 0)
-		(fields_autoplaced yes)
 		(effects
 			(font
@@
 			(justify left)
 		)
-		(property "Netclass" "DP_90R"
-			(at 191.77 44.45 0)
-			(effects
-				(font
-					(size 1.27 1.27)
-					(italic yes)
-				)
-				(justify left)
-				(hide yes)
-			)
-		)
 	)
 	(hierarchical_label "5V"
@@
 		(shape input)
 		(at 82.55 111.76 0)
-		(fields_autoplaced yes)
 		(effects
 			(font
@@
 			(justify left)
 		)
-		(property "Netclass" "DP_90R"
-			(at 82.55 113.03 0)
-			(effects
-				(font
-					(size 1.27 1.27)
-					(italic yes)
-				)
-				(justify left)
-				(hide yes)
-			)
-		)
 	)
 	(hierarchical_label "GPIO45"
@@
 		(shape input)
 		(at 191.77 40.64 0)
-		(fields_autoplaced yes)
 		(effects
 			(font
@@
 			(justify left)
 		)
-		(property "Netclass" "DP_90R"
-			(at 191.77 41.91 0)
-			(effects
-				(font
-					(size 1.27 1.27)
-					(italic yes)
-				)
-				(justify left)
-				(hide yes)
-			)
-		)
 	)
 	(hierarchical_label "GPIO38"
@@
 		(shape input)
 		(at 82.55 114.3 0)
-		(fields_autoplaced yes)
 		(effects
 			(font
@@
 			(justify left)
 		)
-		(property "Netclass" "DP_90R"
-			(at 82.55 115.57 0)
-			(effects
-				(font
-					(size 1.27 1.27)
-					(italic yes)
-				)
-				(justify left)
-				(hide yes)
-			)
-		)
 	)
 	(hierarchical_label "ESP_GND"
@@
 			)
 		)
-		(property "Footprint" "Package_DFN_QFN:QFN-24-1EP_4x4mm_P0.5mm_EP2.7x2.7mm_ThermalVias"
+		(property "Footprint" "yarrboard:QFN-24-1EP_4x4mm_P0.5mm_EP2.7x2.7mm_ThermalVias"
 			(at 172.72 45.72 0)
 			(effects
@@
 			)
 		)
-		(property "Footprint" "Package_DFN_QFN:QFN-16-1EP_3x3mm_P0.5mm_EP1.7x1.7mm_ThermalVias"
+		(property "Footprint" "yarrboard:QFN-16-1EP_3x3mm_P0.5mm_EP1.7x1.7mm_ThermalVias"
 			(at 260.35 66.04 0)
 			(effects
@@
 			)
 		)
-		(property "Footprint" "RF_Module:ESP32-S3-WROOM-1"
+		(property "Footprint" "yarrboard:ESP32-S3-WROOM-1"
 			(at 67.31 121.92 0)
 			(effects

Commit message: worked on bom for rev b prototype run
Parts:
- D20: LCSC (none) -> C191023
- D22: value LED -> RED; LCSC C2286 -> C965799
- Q7: LCSC (none) -> C112086
- R35: value 100 -> 100R
- SW1, SW2: LCSC C843684 -> C557599
- U4: LCSC (none) -> C2913202
- U6: LCSC (none) -> C424705
- U7: LCSC (none) -> C5187527
- U8: LCSC (none) -> C2846043
Changed lines of the file:
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@@
 			)
 		)
+		(property "LCSC" "C5187527"
+			(at 172.72 45.72 0)
+			(effects
+				(font
+					(size 1.27 1.27)
+				)
+				(hide yes)
+			)
+		)
 		(pin "19"
 		)
@@
 			)
 		)
-		(property "Value" "LED"
+		(property "Value" "RED"
 			(at 135.89 118.872 0)
 			(effects
@@
 			)
 		)
-		(property "LCSC" "C2286"
+		(property "LCSC" "C965799"
 			(at 133.35 119.38 0)
 			(effects
@@
 			)
 		)
-		(property "Value" "100"
+		(property "Value" "100R"
 			(at 25.4 182.88 90)
 			(effects
@@
 			)
 		)
+		(property "LCSC" ""
+			(at 229.87 33.02 0)
+			(effects
+				(font
+					(size 1.27 1.27)
+				)
+				(hide yes)
+			)
+		)
 		(pin "1"
 		)
@@
 			)
 		)
+		(property "LCSC" "C2846043"
+			(at 255.27 50.8 0)
+			(effects
+				(font
+					(size 1.27 1.27)
+				)
+				(hide yes)
+			)
+		)
 		(pin "3"
 		)
@@
 			)
 		)
+		(property "LCSC" "C424705"
+			(at 110.49 177.8 0)
+			(effects
+				(font
+					(size 1.27 1.27)
+				)
+				(hide yes)
+			)
+		)
 		(pin "1"
 		)
@@
 			)
 		)
+		(property "LCSC" ""
+			(at 31.75 125.73 0)
+			(effects
+				(font
+					(size 1.27 1.27)
+				)
+				(hide yes)
+			)
+		)
 		(pin "1"
 		)
@@
 			)
 		)
+		(property "LCSC" "C112086"
+			(at 46.99 184.15 0)
+			(effects
+				(font
+					(size 1.27 1.27)
+				)
+				(hide yes)
+			)
+		)
 		(pin "2"
 		)
@@
 			)
 		)
-		(property "LCSC" "C843684"
+		(property "LCSC" "C557599"
 			(at 269.24 110.49 0)
 			(effects
@@
 			)
 		)
+		(property "LCSC" ""
+			(at 218.44 33.02 0)
+			(effects
+				(font
+					(size 1.27 1.27)
+				)
+				(hide yes)
+			)
+		)
 		(pin "1"
 		)
@@
 			)
 		)
+		(property "LCSC" ""
+			(at 72.39 181.61 0)
+			(effects
+				(font
+					(size 1.27 1.27)
+				)
+				(hide yes)
+			)
+		)
 		(pin "1"
 		)
@@
 			)
 		)
-		(property "LCSC" "C843684"
+		(property "LCSC" "C557599"
 			(at 269.24 148.59 0)
 			(effects
@@
 			)
 		)
+		(property "LCSC" ""
+			(at 241.3 33.02 0)
+			(effects
+				(font
+					(size 1.27 1.27)
+				)
+				(hide yes)
+			)
+		)
 		(pin "1"
 		)
@@
 			)
 		)
+		(property "LCSC" ""
+			(at 146.05 181.61 0)
+			(effects
+				(font
+					(size 1.27 1.27)
+				)
+				(hide yes)
+			)
+		)
 		(pin "1"
 		)
@@
 			)
 		)
+		(property "LCSC" ""
+			(at 161.29 146.05 0)
+			(effects
+				(font
+					(size 1.27 1.27)
+				)
+				(hide yes)
+			)
+		)
 		(pin "1"
 		)
@@
 			)
 		)
+		(property "LCSC" "C2913202"
+			(at 67.31 124.46 0)
+			(effects
+				(font
+					(size 1.27 1.27)
+				)
+				(hide yes)
+			)
+		)
 		(pin "1"
 		)
@@
 			)
 		)
+		(property "LCSC" ""
+			(at 231.14 45.72 90)
+			(effects
+				(font
+					(size 1.27 1.27)
+				)
+				(hide yes)
+			)
+		)
 		(pin "1"
 		)
@@
 			)
 		)
+		(property "LCSC" "C191023"
+			(at 59.69 33.02 0)
+			(effects
+				(font
+					(size 1.27 1.27)
+				)
+				(hide yes)
+			)
+		)

Commit message: updated jlc parts rotations and placement offsets
Parts:
- J18: Position Offset (none) -> 0.0,1.27
- SW1, SW2, U7, U8: Rotation Offset (none) -> 180
- U4: Position Offset (none) -> 0,-3.6195
- U5: Rotation Offset (none) -> 90
Changed lines of the file:
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@@
+			)
+		)
+		(property "Rotation Offset" "180"
+			(at 172.72 45.72 0)
+			(effects
+				(font
+					(size 1.27 1.27)
+				)
+				(hide yes)
 			)
 		)
@@
 		)
 		(property "LCSC" "C2846043"
+			(at 255.27 50.8 0)
+			(effects
+				(font
+					(size 1.27 1.27)
+				)
+				(hide yes)
+			)
+		)
+		(property "Rotation Offset" "180"
 			(at 255.27 50.8 0)
 			(effects
@@
 			)
 		)
+		(property "Rotation Offset" "90"
+			(at 73.66 67.31 0)
+			(effects
+				(font
+					(size 1.27 1.27)
+				)
+				(hide yes)
+			)
+		)
 		(pin "1"
 		)
@@
 			)
 		)
+		(property "Rotation Offset" "180"
+			(at 269.24 110.49 0)
+			(effects
+				(font
+					(size 1.27 1.27)
+				)
+				(hide yes)
+			)
+		)
 		(pin "1"
 		)
@@
 			)
 		)
+		(property "Rotation Offset" "180"
+			(at 269.24 148.59 0)
+			(effects
+				(font
+					(size 1.27 1.27)
+				)
+				(hide yes)
+			)
+		)
 		(pin "1"
 		)
@@
 			)
 		)
+		(property "Position Offset" "0,-3.6195"
+			(at 67.31 124.46 0)
+			(effects
+				(font
+					(size 1.27 1.27)
+				)
+				(hide yes)
+			)
+		)
 		(pin "1"
 		)
@@
 			(at 29.21 48.26 0)
 			(effects
+				(font
+					(size 1.27 1.27)
+				)
+				(hide yes)
+			)
+		)
+		(property "Position Offset" "0.0,1.27"
+			(at 29.21 48.26 0)
+			(effects

Commit message: copied back from esp32-s3-template
Parts:
- renumbered C15 to C1, C24 to C10, C25 to C11, C26 to C12, C27 to C13, C28 to C14, C29 to C15, C30 to C16, C31 to C17, C32 to C18, C33 to C19, C16 to C2, C17 to C3, C18 to C4, C19 to C5, C20 to C6, C21 to C7, C22 to C8, C23 to C9, D20 to D1, D22 to D2, D21 to D3, FB2 to FB1, J18 to J3, Q7 to Q1, Q8 to Q2, Q9 to Q3, R35 to R1, R44 to R10, R45 to R11, R36 to R2, R37 to R3, R38 to R4, R39 to R5, R41 to R6, R40 to R7, R42 to R8, R43 to R9, U4 to U1, U5 to U2, U6 to U3, U7 to U4, U8 to U5
Other:
- moved on the sheet: D2, R6
