File: brineomatic/rs485.kicad_sch (KiCad schematic)
At the start: 13 parts, among them J22 3.5mm, J23 3.5mm, U10 MAX3485

Commit message: removed rs485 jumper and added silkscreen
Parts:
- removed JP1: SolderJumper_2_Bridged, Jumper:SolderJumper-2_P1.3mm_Bridged_RoundedPad1.0x1.5mm, symbol Jumper:SolderJumper_2_Bridged
- J22: footprint Connector_Phoenix_MC:PhoenixContact_MC_1,5_3-G-3.5_1x03_P3.50mm_Horizontal -> yarrboard:PhoenixContact_MC_1,5_3-G-3.5_1x03_P3.50mm_Horizontal
Connections:
- net at R54.2: now also J22.1 (Pin_1), R52.1, U10.6 (A)
Other:
- moved on the sheet: R54
Changed lines of the file:
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@@
+	)
+	(junction
+		(at 171.45 93.98)
+		(diameter 0)
+		(color 0 0 0 0)
+	)
+	(junction
+		(at 171.45 99.06)
+		(diameter 0)
+		(color 0 0 0 0)
 	)
 	(junction
@@
 	)
 	(junction
-		(at 171.45 93.98)
-		(diameter 0)
-		(color 0 0 0 0)
-	)
-	(junction
-		(at 160.02 107.95)
-		(diameter 0)
-		(color 0 0 0 0)
-	)
-	(junction
 		(at 123.19 82.55)
 		(diameter 0)
@@
 	)
 	(junction
-		(at 171.45 107.95)
-		(diameter 0)
-		(color 0 0 0 0)
-	)
-	(junction
 		(at 160.02 93.98)
 		(diameter 0)
@@
 	)
 	(junction
+		(at 160.02 99.06)
+		(diameter 0)
+		(color 0 0 0 0)
+	)
+	(junction
 		(at 114.3 82.55)
 		(diameter 0)
@@
 	(wire
 		(pts
-			(xy 171.45 107.95) (xy 181.61 107.95)
+			(xy 171.45 99.06) (xy 181.61 99.06)
 		)
 		(stroke
@@
 	(wire
 		(pts
-			(xy 160.02 107.95) (xy 160.02 111.76)
+			(xy 171.45 93.98) (xy 186.69 93.98)
 		)
 		(stroke
@@
 	(wire
 		(pts
-			(xy 171.45 107.95) (xy 171.45 106.68)
-		)
-		(stroke
-			(width 0)
-			(type default)
-		)
-	)
-	(wire
-		(pts
 			(xy 83.82 82.55) (xy 72.39 82.55)
 		)
@@
 	(wire
 		(pts
-			(xy 171.45 93.98) (xy 186.69 93.98)
+			(xy 160.02 93.98) (xy 171.45 93.98)
 		)
 		(stroke
@@
 	(wire
 		(pts
-			(xy 160.02 107.95) (xy 171.45 107.95)
+			(xy 160.02 99.06) (xy 171.45 99.06)
 		)
 		(stroke
@@
 	(wire
 		(pts
-			(xy 160.02 93.98) (xy 171.45 93.98)
+			(xy 160.02 99.06) (xy 160.02 111.76)
 		)
 		(stroke
@@
 	(wire
 		(pts
-			(xy 181.61 107.95) (xy 181.61 96.52)
+			(xy 181.61 99.06) (xy 181.61 96.52)
 		)
 		(stroke
@@
 		(pts
 			(xy 186.69 123.19) (xy 160.02 123.19)
-		)
-		(stroke
-			(width 0)
-			(type default)
-		)
-	)
-	(wire
-		(pts
-			(xy 160.02 99.06) (xy 160.02 107.95)
 		)
 		(stroke
@@
 	)
 	(symbol
-		(lib_id "Jumper:SolderJumper_2_Bridged")
-		(at 171.45 97.79 90)
-		(unit 1)
-		(exclude_from_sim no)
-		(in_bom no)
-		(on_board yes)
-		(dnp no)
-		(fields_autoplaced yes)
-		(property "Reference" "JP1"
-			(at 173.99 96.5199 90)
-			(effects
-				(font
-					(size 1.27 1.27)
-				)
-				(justify right)
-			)
-		)
-		(property "Value" "SolderJumper_2_Bridged"
-			(at 173.99 99.0599 90)
-			(effects
-				(font
-					(size 1.27 1.27)
-				)
-				(justify right)
-				(hide yes)
-			)
-		)
-		(property "Footprint" "Jumper:SolderJumper-2_P1.3mm_Bridged_RoundedPad1.0x1.5mm"
-			(at 171.45 97.79 0)
-			(effects
-				(font
-					(size 1.27 1.27)
-				)
-				(hide yes)
-			)
-		)
-		(property "Datasheet" "~"
-			(at 171.45 97.79 0)
-			(effects
-				(font
-					(size 1.27 1.27)
-				)
-				(hide yes)
-			)
-		)
-		(property "Description" "Solder Jumper, 2-pole, closed/bridged"
-			(at 171.45 97.79 0)
-			(effects
-				(font
-					(size 1.27 1.27)
-				)
-				(hide yes)
-			)
-		)
-		(pin "2"
-		)
-		(pin "1"
-		)
-		(instances
-			(project ""
-				(path "/96477ae2-ef08-48f3-8dd4-fe4478541f68/ecabf60a-7f79-4ba0-9fc6-a1e702c2d5f0"
-					(reference "JP1")
-					(unit 1)
-				)
-			)
-		)
-	)
-	(symbol
 		(lib_id "Device:C_Small")
 		(at 72.39 101.6 0)
@@
 	(symbol
 		(lib_id "Device:R_Small_US")
-		(at 171.45 104.14 180)
+		(at 171.45 96.52 180)
 		(unit 1)
 		(exclude_from_sim no)
@@
 		(dnp no)
 		(property "Reference" "R54"
-			(at 173.228 103.124 0)
+			(at 173.228 95.504 0)
 			(effects
 				(font
@@
 		)
 		(property "Value" "120R"
-			(at 173.228 105.664 0)
+			(at 173.228 98.044 0)
 			(effects
 				(font
@@
 		)
 		(property "Footprint" "Resistor_SMD:R_0603_1608Metric"
-			(at 171.45 104.14 0)
+			(at 171.45 96.52 0)
 			(effects
 				(font
@@
 		)
 		(property "Datasheet" "~"
-			(at 171.45 104.14 0)
+			(at 171.45 96.52 0)
 			(effects
 				(font
@@
 		)
 		(property "Description" "Resistor, small US symbol"
-			(at 171.45 104.14 0)
+			(at 171.45 96.52 0)
 			(effects
 				(font
@@
 			)
 		)
-		(property "Footprint" "Connector_Phoenix_MC:PhoenixContact_MC_1,5_3-G-3.5_1x03_P3.50mm_Horizontal"
+		(property "Footprint" "yarrboard:PhoenixContact_MC_1,5_3-G-3.5_1x03_P3.50mm_Horizontal"
 			(at 191.77 96.52 0)
 			(effects

Commit message: added back up usb serial converter headers
Parts:
- renumbered J22 to J23, J23 to J24
Changed lines of the file:
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@@
 		(dnp no)
 		(fields_autoplaced yes)
-		(property "Reference" "#PWR068"
+		(property "Reference" "#PWR070"
 			(at 140.97 130.81 0)
 			(effects
@@
 			(project "brineomatic"
 				(path "/96477ae2-ef08-48f3-8dd4-fe4478541f68/ecabf60a-7f79-4ba0-9fc6-a1e702c2d5f0"
-					(reference "#PWR068")
+					(reference "#PWR070")
 					(unit 1)
 				)
@@
 		(dnp no)
 		(fields_autoplaced yes)
-		(property "Reference" "#PWR067"
+		(property "Reference" "#PWR069"
 			(at 140.97 83.82 0)
 			(effects
@@
 			(project ""
 				(path "/96477ae2-ef08-48f3-8dd4-fe4478541f68/ecabf60a-7f79-4ba0-9fc6-a1e702c2d5f0"
-					(reference "#PWR067")
+					(reference "#PWR069")
 					(unit 1)
 				)
@@
 		(dnp no)
 		(fields_autoplaced yes)
-		(property "Reference" "J22"
+		(property "Reference" "J23"
 			(at 194.31 95.2499 0)
 			(effects
@@
 			(project ""
 				(path "/96477ae2-ef08-48f3-8dd4-fe4478541f68/ecabf60a-7f79-4ba0-9fc6-a1e702c2d5f0"
-					(reference "J22")
+					(reference "J23")
 					(unit 1)
 				)
@@
 		(dnp no)
 		(fields_autoplaced yes)
-		(property "Reference" "J23"
+		(property "Reference" "J24"
 			(at 210.82 95.2499 0)
 			(effects
@@
 			(project ""
 				(path "/96477ae2-ef08-48f3-8dd4-fe4478541f68/ecabf60a-7f79-4ba0-9fc6-a1e702c2d5f0"
-					(reference "J23")
-					(unit 1)
-				)
+					(reference "J24")
+					(unit 1)
+				)

Commit message: switched to the LDL1117 ldo
Parts:
- renumbered C36 to C35, C37 to C36, R48 to R47, R49 to R48, R50 to R49, R51 to R50, R52 to R51, R53 to R52, R54 to R53
Changed lines of the file:
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@@
 		(on_board yes)
 		(dnp no)
-		(property "Reference" "R53"
+		(property "Reference" "R52"
 			(at 161.798 113.284 0)
 			(effects
@@
 			(project "brineomatic"
 				(path "/96477ae2-ef08-48f3-8dd4-fe4478541f68/ecabf60a-7f79-4ba0-9fc6-a1e702c2d5f0"
-					(reference "R53")
+					(reference "R52")
 					(unit 1)
 				)
@@
 		(on_board yes)
 		(dnp no)
-		(property "Reference" "R48"
+		(property "Reference" "R47"
 			(at 98.298 90.424 0)
 			(effects
@@
 			(project "brineomatic"
 				(path "/96477ae2-ef08-48f3-8dd4-fe4478541f68/ecabf60a-7f79-4ba0-9fc6-a1e702c2d5f0"
-					(reference "R48")
+					(reference "R47")
 					(unit 1)
 				)
@@
 		(on_board yes)
 		(dnp no)
-		(property "Reference" "C36"
+		(property "Reference" "C35"
 			(at 74.93 100.3363 0)
 			(effects
@@
 			(project "brineomatic"
 				(path "/96477ae2-ef08-48f3-8dd4-fe4478541f68/ecabf60a-7f79-4ba0-9fc6-a1e702c2d5f0"
-					(reference "C36")
+					(reference "C35")
 					(unit 1)
 				)
@@
 		(on_board yes)
 		(dnp no)
-		(property "Reference" "R50"
+		(property "Reference" "R49"
 			(at 116.078 90.424 0)
 			(effects
@@
 			(project "brineomatic"
 				(path "/96477ae2-ef08-48f3-8dd4-fe4478541f68/ecabf60a-7f79-4ba0-9fc6-a1e702c2d5f0"
-					(reference "R50")
+					(reference "R49")
 					(unit 1)
 				)
@@
 		(on_board yes)
 		(dnp no)
-		(property "Reference" "R51"
+		(property "Reference" "R50"
 			(at 124.968 90.424 0)
 			(effects
@@
 			(project "brineomatic"
 				(path "/96477ae2-ef08-48f3-8dd4-fe4478541f68/ecabf60a-7f79-4ba0-9fc6-a1e702c2d5f0"
-					(reference "R51")
+					(reference "R50")
 					(unit 1)
 				)
@@
 		(on_board yes)
 		(dnp no)
-		(property "Reference" "R54"
+		(property "Reference" "R53"
 			(at 173.228 95.504 0)
 			(effects
@@
 			(project "brineomatic"
 				(path "/96477ae2-ef08-48f3-8dd4-fe4478541f68/ecabf60a-7f79-4ba0-9fc6-a1e702c2d5f0"
-					(reference "R54")
+					(reference "R53")
 					(unit 1)
 				)
@@
 		(dnp no)
 		(fields_autoplaced yes)
-		(property "Reference" "C37"
+		(property "Reference" "C36"
 			(at 86.36 100.3363 0)
 			(effects
@@
 			(project "brineomatic"
 				(path "/96477ae2-ef08-48f3-8dd4-fe4478541f68/ecabf60a-7f79-4ba0-9fc6-a1e702c2d5f0"
-					(reference "C37")
+					(reference "C36")
 					(unit 1)
 				)
@@
 		(on_board yes)
 		(dnp no)
-		(property "Reference" "R49"
+		(property "Reference" "R48"
 			(at 107.188 90.424 0)
 			(effects
@@
 			(project "brineomatic"
 				(path "/96477ae2-ef08-48f3-8dd4-fe4478541f68/ecabf60a-7f79-4ba0-9fc6-a1e702c2d5f0"
-					(reference "R49")
+					(reference "R48")
 					(unit 1)
 				)
@@
 		(on_board yes)
 		(dnp no)
-		(property "Reference" "R52"
+		(property "Reference" "R51"
 			(at 161.798 86.614 0)
 			(effects
@@
 			(project "brineomatic"
 				(path "/96477ae2-ef08-48f3-8dd4-fe4478541f68/ecabf60a-7f79-4ba0-9fc6-a1e702c2d5f0"
-					(reference "R52")
-					(unit 1)
-				)
+					(reference "R51")
+					(unit 1)
+				)
