File: brineomatic/tds.kicad_sch (KiCad schematic)
At the start: 4 parts

Commit message: switched to bav199 on pressure / tds
Parts:
- C3: value 1uF -> 100nF
- D7: value BAT54S -> BAV199; LCSC C727126 -> C40919
- R9: value 1k -> 10k
Changed lines of the file:
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@@
 			)
 		)
-		(property "Value" "1k"
+		(property "Value" "10k"
 			(at 111.76 82.804 90)
 			(effects
@@
 			)
 		)
-		(property "Value" "1uF"
+		(property "Value" "100nF"
 			(at 120.65 90.1763 0)
 			(effects
@@
 			)
 		)
-		(property "Value" "BAT54S"
+		(property "Value" "BAV199"
 			(at 133.35 86.36 90)
 			(effects
@@
 			)
 		)
-		(property "Datasheet" "https://www.diodes.com/assets/Datasheets/ds11005.pdf"
+		(property "Datasheet" "https://www.lcsc.com/datasheet/C40919.pdf"
 			(at 130.81 88.138 0)
 			(effects
@@
 			)
 		)
-		(property "LCSC" "C727126"
+		(property "LCSC" "C40919"
 			(at 130.81 85.09 90)
 			(effects

Commit message: tested and update bom + placement
Parts:
- C3: LCSC (none) -> C14663
Changed lines of the file:
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@@
 			)
 		)
-		(property "LCSC" ""
+		(property "LCSC" "C14663"
 			(at 118.11 88.9 0)
 			(effects

Commit message: updated resistor p/ns in bom
Parts:
- R9: LCSC (none) -> C25804
Changed lines of the file:
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@@
 			)
 		)
-		(property "LCSC" ""
+		(property "LCSC" "C25804"
 			(at 111.76 85.09 0)
 			(effects

Commit message: add inline resistor to temperature sensor + servo inputs - 100ohm
Parts:
- renumbered R9 to R10
Changed lines of the file:
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@@
 		(on_board yes)
 		(dnp no)
-		(property "Reference" "R9"
+		(property "Reference" "R10"
 			(at 111.76 80.518 90)
 			(effects
@@
 			(project "brineomatic"
 				(path "/96477ae2-ef08-48f3-8dd4-fe4478541f68/4dde40bf-0b86-4621-acd9-eb6c6b71c357"
-					(reference "R51")
+					(reference "R54")
 					(unit 1)
 				)
 				(path "/96477ae2-ef08-48f3-8dd4-fe4478541f68/be3403ab-9eef-436c-86e7-0de3f072ae30"
-					(reference "R9")
+					(reference "R10")
 					(unit 1)
 				)
