File: brineomatic/1115_adc.kicad_sch (KiCad schematic)
At the start: 10 parts, among them U1 ADS1115IDGSR

Commit message: added more esd protection to the power rails (24v, 5v, 3.3v)
Parts:
- D13: renamed from D12; LCSC (none) -> C2687129
- D14: renamed from D13; LCSC (none) -> C2687129
Changed lines of the file:
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@@
 		(on_board yes)
 		(dnp no)
-		(property "Reference" "D12"
+		(property "Reference" "D13"
 			(at 175.26 93.9799 90)
 			(effects
@@
 		)
 		(property "Supplier Part" ""
+			(at 177.8 95.25 90)
+			(effects
+				(font
+					(size 1.27 1.27)
+				)
+				(hide yes)
+			)
+		)
+		(property "LCSC" "C2687129"
 			(at 177.8 95.25 90)
 			(effects
@@
 			(project "brineomatic"
 				(path "/96477ae2-ef08-48f3-8dd4-fe4478541f68/64f85b9c-b5dc-4ec9-9075-ce977ed1cba6"
-					(reference "D12")
+					(reference "D13")
 					(unit 1)
 				)
@@
 		(on_board yes)
 		(dnp no)
-		(property "Reference" "D13"
+		(property "Reference" "D14"
 			(at 190.5 93.9799 90)
 			(effects
@@
 		)
 		(property "Supplier Part" ""
+			(at 187.96 95.25 90)
+			(effects
+				(font
+					(size 1.27 1.27)
+				)
+				(hide yes)
+			)
+		)
+		(property "LCSC" "C2687129"
 			(at 187.96 95.25 90)
 			(effects
@@
 			(project "brineomatic"
 				(path "/96477ae2-ef08-48f3-8dd4-fe4478541f68/64f85b9c-b5dc-4ec9-9075-ce977ed1cba6"
-					(reference "D13")
+					(reference "D14")
 					(unit 1)
 				)

Commit message: tested and update bom + placement
Parts:
- C4: LCSC (none) -> C14663
Changed lines of the file:
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@@
 			)
 		)
-		(property "LCSC" ""
+		(property "LCSC" "C14663"
 			(at 204.47 81.28 0)
 			(effects

Commit message: updated resistor p/ns in bom
Parts:
- R13: LCSC (none) -> C25804
- R14, R15: LCSC (none) -> C4190
- U1: Mouser 595-ADS1115IDGSR -> (none)
Changed lines of the file:
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@@
 			)
 		)
-		(property "LCSC" ""
+		(property "LCSC" " C4190"
 			(at 177.8 81.28 0)
 			(effects
@@
 			)
 		)
-		(property "Mouser" " 595-ADS1115IDGSR "
+		(property "Mouser" ""
 			(at 127 86.36 0)
 			(effects
@@
 			)
 		)
+		(property "LCSC" "C25804"
+			(at 148.59 74.93 0)
+			(effects
+				(font
+					(size 1.27 1.27)
+				)
+				(hide yes)
+			)
+		)
 		(pin "1"
 		)
@@
 			)
 		)
-		(property "LCSC" ""
+		(property "LCSC" " C4190"
 			(at 187.96 81.28 0)
 			(effects

Commit message: added esd protection to relay driver connector
Parts:
- renumbered C4 to C6, C5 to C7, D13 to D14, D14 to D15
Changed lines of the file:
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@@
 		(on_board yes)
 		(dnp no)
-		(property "Reference" "C4"
+		(property "Reference" "C6"
 			(at 207.01 80.0163 0)
 			(effects
@@
 			(project "brineomatic"
 				(path "/96477ae2-ef08-48f3-8dd4-fe4478541f68/64f85b9c-b5dc-4ec9-9075-ce977ed1cba6"
-					(reference "C4")
+					(reference "C6")
 					(unit 1)
 				)
@@
 		(on_board yes)
 		(dnp no)
-		(property "Reference" "C5"
+		(property "Reference" "C7"
 			(at 218.44 80.0163 0)
 			(effects
@@
 			(project "brineomatic"
 				(path "/96477ae2-ef08-48f3-8dd4-fe4478541f68/64f85b9c-b5dc-4ec9-9075-ce977ed1cba6"
-					(reference "C5")
+					(reference "C7")
 					(unit 1)
 				)
@@
 		(on_board yes)
 		(dnp no)
-		(property "Reference" "D13"
+		(property "Reference" "D14"
 			(at 175.26 93.9799 90)
 			(effects
@@
 			(project "brineomatic"
 				(path "/96477ae2-ef08-48f3-8dd4-fe4478541f68/64f85b9c-b5dc-4ec9-9075-ce977ed1cba6"
-					(reference "D13")
+					(reference "D14")
 					(unit 1)
 				)
@@
 		(on_board yes)
 		(dnp no)
-		(property "Reference" "D14"
+		(property "Reference" "D15"
 			(at 190.5 93.9799 90)
 			(effects
@@
 			(project "brineomatic"
 				(path "/96477ae2-ef08-48f3-8dd4-fe4478541f68/64f85b9c-b5dc-4ec9-9075-ce977ed1cba6"
-					(reference "D14")
+					(reference "D15")
 					(unit 1)
 				)

Commit message: add inline resistor to temperature sensor + servo inputs - 100ohm
Parts:
- renumbered R13 to R16, R14 to R17, R15 to R18
Changed lines of the file:
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@@
 		(dnp no)
 		(fields_autoplaced yes)
-		(property "Reference" "R14"
+		(property "Reference" "R17"
 			(at 180.34 80.0099 0)
 			(effects
@@
 			(project "brineomatic"
 				(path "/96477ae2-ef08-48f3-8dd4-fe4478541f68/64f85b9c-b5dc-4ec9-9075-ce977ed1cba6"
-					(reference "R14")
+					(reference "R17")
 					(unit 1)
 				)
@@
 		(dnp no)
 		(fields_autoplaced yes)
-		(property "Reference" "R13"
+		(property "Reference" "R16"
 			(at 151.13 73.6599 0)
 			(effects
@@
 			(project "brineomatic"
 				(path "/96477ae2-ef08-48f3-8dd4-fe4478541f68/64f85b9c-b5dc-4ec9-9075-ce977ed1cba6"
-					(reference "R13")
+					(reference "R16")
 					(unit 1)
 				)
@@
 		(dnp no)
 		(fields_autoplaced yes)
-		(property "Reference" "R15"
+		(property "Reference" "R18"
 			(at 190.5 80.0099 0)
 			(effects
@@
 			(project "brineomatic"
 				(path "/96477ae2-ef08-48f3-8dd4-fe4478541f68/64f85b9c-b5dc-4ec9-9075-ce977ed1cba6"
-					(reference "R15")
+					(reference "R18")
 					(unit 1)
 				)

Commit message: updated analog sensor esd schematic
Parts:
- renumbered D14 to D15, D15 to D16
Changed lines of the file:
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@@
 		(dnp no)
 		(fields_autoplaced yes)
-		(property "Reference" "#PWR022"
+		(property "Reference" "#PWR023"
 			(at 127 69.85 0)
 			(effects
@@
 			(project "brineomatic"
 				(path "/96477ae2-ef08-48f3-8dd4-fe4478541f68/64f85b9c-b5dc-4ec9-9075-ce977ed1cba6"
-					(reference "#PWR022")
+					(reference "#PWR023")
 					(unit 1)
 				)
@@
 		(on_board yes)
 		(dnp no)
-		(property "Reference" "D14"
+		(property "Reference" "D15"
 			(at 175.26 93.9799 90)
 			(effects
@@
 			(project "brineomatic"
 				(path "/96477ae2-ef08-48f3-8dd4-fe4478541f68/64f85b9c-b5dc-4ec9-9075-ce977ed1cba6"
-					(reference "D14")
+					(reference "D15")
 					(unit 1)
 				)
@@
 		(on_board yes)
 		(dnp no)
-		(property "Reference" "D15"
+		(property "Reference" "D16"
 			(at 190.5 93.9799 90)
 			(effects
@@
 			(project "brineomatic"
 				(path "/96477ae2-ef08-48f3-8dd4-fe4478541f68/64f85b9c-b5dc-4ec9-9075-ce977ed1cba6"
-					(reference "D15")
+					(reference "D16")
 					(unit 1)
 				)
@@
 		(dnp no)
 		(fields_autoplaced yes)
-		(property "Reference" "#PWR023"
+		(property "Reference" "#PWR024"
 			(at 127 105.41 0)
 			(effects
@@
 			(project ""
 				(path "/96477ae2-ef08-48f3-8dd4-fe4478541f68/64f85b9c-b5dc-4ec9-9075-ce977ed1cba6"
-					(reference "#PWR023")
+					(reference "#PWR024")
 					(unit 1)
 				)

Commit message: added bulk cap after ideal diode
Parts:
- renumbered D15 to D16, D16 to D17
Changed lines of the file:
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@@
 		(dnp no)
 		(fields_autoplaced yes)
-		(property "Reference" "#PWR023"
+		(property "Reference" "#PWR025"
 			(at 127 69.85 0)
 			(effects
@@
 			(project "brineomatic"
 				(path "/96477ae2-ef08-48f3-8dd4-fe4478541f68/64f85b9c-b5dc-4ec9-9075-ce977ed1cba6"
-					(reference "#PWR023")
+					(reference "#PWR025")
 					(unit 1)
 				)
@@
 		(on_board yes)
 		(dnp no)
-		(property "Reference" "D15"
+		(property "Reference" "D16"
 			(at 175.26 93.9799 90)
 			(effects
@@
 			(project "brineomatic"
 				(path "/96477ae2-ef08-48f3-8dd4-fe4478541f68/64f85b9c-b5dc-4ec9-9075-ce977ed1cba6"
-					(reference "D15")
+					(reference "D16")
 					(unit 1)
 				)
@@
 		(on_board yes)
 		(dnp no)
-		(property "Reference" "D16"
+		(property "Reference" "D17"
 			(at 190.5 93.9799 90)
 			(effects
@@
 			(project "brineomatic"
 				(path "/96477ae2-ef08-48f3-8dd4-fe4478541f68/64f85b9c-b5dc-4ec9-9075-ce977ed1cba6"
-					(reference "D16")
+					(reference "D17")
 					(unit 1)
 				)
@@
 		(dnp no)
 		(fields_autoplaced yes)
-		(property "Reference" "#PWR024"
+		(property "Reference" "#PWR026"
 			(at 127 105.41 0)
 			(effects
@@
 			(project ""
 				(path "/96477ae2-ef08-48f3-8dd4-fe4478541f68/64f85b9c-b5dc-4ec9-9075-ce977ed1cba6"
-					(reference "#PWR024")
+					(reference "#PWR026")
 					(unit 1)
 				)
