File: brineomatic/tmc2209.kicad_sch (KiCad schematic)
At the start: 21 parts, among them J21 Conn_01x04, U9 TMC2209-LA

Commit message: added more input/output caps
Parts:
- renumbered C36 to C38, C37 to C39, C38 to C40, C39 to C41, C40 to C42, C41 to C43, C43 to C45, C44 to C46, C45 to C47, C46 to C48, C47 to C49, C48 to C50, C49 to C51
Changed lines of the file:
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@@
 		(on_board yes)
 		(dnp no)
-		(property "Reference" "C41"
+		(property "Reference" "C43"
 			(at 118.11 45.72 0)
 			(effects
@@
 			(project "brineomatic"
 				(path "/96477ae2-ef08-48f3-8dd4-fe4478541f68/0f01c39f-0c25-414e-9ed3-1ba09e2af0c5"
-					(reference "C41")
+					(reference "C43")
 					(unit 1)
 				)
@@
 		(on_board yes)
 		(dnp no)
-		(property "Reference" "C46"
+		(property "Reference" "C48"
 			(at 148.59 45.974 0)
 			(effects
@@
 			(project "brineomatic"
 				(path "/96477ae2-ef08-48f3-8dd4-fe4478541f68/0f01c39f-0c25-414e-9ed3-1ba09e2af0c5"
-					(reference "C46")
+					(reference "C48")
 					(unit 1)
 				)
@@
 		(on_board yes)
 		(dnp no)
-		(property "Reference" "C37"
+		(property "Reference" "C39"
 			(at 84.074 62.738 90)
 			(effects
@@
 			(project "brineomatic"
 				(path "/96477ae2-ef08-48f3-8dd4-fe4478541f68/0f01c39f-0c25-414e-9ed3-1ba09e2af0c5"
-					(reference "C37")
+					(reference "C39")
 					(unit 1)
 				)
@@
 		(on_board yes)
 		(dnp no)
-		(property "Reference" "C47"
+		(property "Reference" "C49"
 			(at 151.384 96.52 90)
 			(effects
@@
 			(project "brineomatic"
 				(path "/96477ae2-ef08-48f3-8dd4-fe4478541f68/0f01c39f-0c25-414e-9ed3-1ba09e2af0c5"
-					(reference "C47")
+					(reference "C49")
 					(unit 1)
 				)
@@
 		(on_board yes)
 		(dnp no)
-		(property "Reference" "C45"
+		(property "Reference" "C47"
 			(at 141.224 127 90)
 			(effects
@@
 			(project "brineomatic"
 				(path "/96477ae2-ef08-48f3-8dd4-fe4478541f68/0f01c39f-0c25-414e-9ed3-1ba09e2af0c5"
-					(reference "C45")
+					(reference "C47")
 					(unit 1)
 				)
@@
 		(on_board yes)
 		(dnp no)
-		(property "Reference" "C49"
+		(property "Reference" "C51"
 			(at 163.83 46.99 0)
 			(effects
@@
 			(project ""
 				(path "/96477ae2-ef08-48f3-8dd4-fe4478541f68/0f01c39f-0c25-414e-9ed3-1ba09e2af0c5"
-					(reference "C49")
+					(reference "C51")
 					(unit 1)
 				)
@@
 		(on_board yes)
 		(dnp no)
-		(property "Reference" "C38"
+		(property "Reference" "C40"
 			(at 100.838 45.72 0)
 			(effects
@@
 			(project "brineomatic"
 				(path "/96477ae2-ef08-48f3-8dd4-fe4478541f68/0f01c39f-0c25-414e-9ed3-1ba09e2af0c5"
-					(reference "C38")
+					(reference "C40")
 					(unit 1)
 				)
@@
 		(on_board yes)
 		(dnp no)
-		(property "Reference" "C44"
+		(property "Reference" "C46"
 			(at 141.224 96.52 90)
 			(effects
@@
 			(project "brineomatic"
 				(path "/96477ae2-ef08-48f3-8dd4-fe4478541f68/0f01c39f-0c25-414e-9ed3-1ba09e2af0c5"
-					(reference "C44")
+					(reference "C46")
 					(unit 1)
 				)
@@
 		(on_board yes)
 		(dnp no)
-		(property "Reference" "C48"
+		(property "Reference" "C50"
 			(at 151.384 127 90)
 			(effects
@@
 			(project "brineomatic"
 				(path "/96477ae2-ef08-48f3-8dd4-fe4478541f68/0f01c39f-0c25-414e-9ed3-1ba09e2af0c5"
-					(reference "C48")
+					(reference "C50")
 					(unit 1)
 				)
@@
 		(on_board yes)
 		(dnp no)
-		(property "Reference" "C36"
+		(property "Reference" "C38"
 			(at 66.04 63.754 0)
 			(effects
@@
 			(project "brineomatic"
 				(path "/96477ae2-ef08-48f3-8dd4-fe4478541f68/0f01c39f-0c25-414e-9ed3-1ba09e2af0c5"
-					(reference "C36")
+					(reference "C38")
 					(unit 1)
 				)
@@
 		(on_board yes)
 		(dnp no)
-		(property "Reference" "C40"
+		(property "Reference" "C42"
 			(at 104.14 92.964 90)
 			(effects
@@
 			(project "brineomatic"
 				(path "/96477ae2-ef08-48f3-8dd4-fe4478541f68/0f01c39f-0c25-414e-9ed3-1ba09e2af0c5"
-					(reference "C40")
+					(reference "C42")
 					(unit 1)
 				)
@@
 		(on_board yes)
 		(dnp no)
-		(property "Reference" "C39"
+		(property "Reference" "C41"
 			(at 104.14 81.28 90)
 			(effects
@@
 			(project "brineomatic"
 				(path "/96477ae2-ef08-48f3-8dd4-fe4478541f68/0f01c39f-0c25-414e-9ed3-1ba09e2af0c5"
-					(reference "C39")
+					(reference "C41")
 					(unit 1)
 				)
@@
 		(on_board yes)
 		(dnp no)
-		(property "Reference" "C43"
+		(property "Reference" "C45"
 			(at 130.556 45.974 0)
 			(effects
@@
 			(project "brineomatic"
 				(path "/96477ae2-ef08-48f3-8dd4-fe4478541f68/0f01c39f-0c25-414e-9ed3-1ba09e2af0c5"
-					(reference "C43")
-					(unit 1)
-				)
+					(reference "C45")
+					(unit 1)
+				)

Commit message: added 1uF cap to pressure sensor connectors for esd
Parts:
- renumbered C38 to C40, C39 to C41, C40 to C42, C41 to C43, C42 to C44, C43 to C45, C45 to C47, C46 to C48, C47 to C49, C48 to C50, C49 to C51, C50 to C52, C51 to C53
Changed lines of the file:
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@@
 		(on_board yes)
 		(dnp no)
-		(property "Reference" "C43"
+		(property "Reference" "C45"
 			(at 118.11 45.72 0)
 			(effects
@@
 			(project "brineomatic"
 				(path "/96477ae2-ef08-48f3-8dd4-fe4478541f68/0f01c39f-0c25-414e-9ed3-1ba09e2af0c5"
-					(reference "C43")
+					(reference "C45")
 					(unit 1)
 				)
@@
 		(on_board yes)
 		(dnp no)
-		(property "Reference" "C48"
+		(property "Reference" "C50"
 			(at 148.59 45.974 0)
 			(effects
@@
 			(project "brineomatic"
 				(path "/96477ae2-ef08-48f3-8dd4-fe4478541f68/0f01c39f-0c25-414e-9ed3-1ba09e2af0c5"
-					(reference "C48")
+					(reference "C50")
 					(unit 1)
 				)
@@
 		(on_board yes)
 		(dnp no)
-		(property "Reference" "C39"
+		(property "Reference" "C41"
 			(at 84.074 62.738 90)
 			(effects
@@
 			(project "brineomatic"
 				(path "/96477ae2-ef08-48f3-8dd4-fe4478541f68/0f01c39f-0c25-414e-9ed3-1ba09e2af0c5"
-					(reference "C39")
+					(reference "C41")
 					(unit 1)
 				)
@@
 		(on_board yes)
 		(dnp no)
-		(property "Reference" "C49"
+		(property "Reference" "C51"
 			(at 151.384 96.52 90)
 			(effects
@@
 			(project "brineomatic"
 				(path "/96477ae2-ef08-48f3-8dd4-fe4478541f68/0f01c39f-0c25-414e-9ed3-1ba09e2af0c5"
-					(reference "C49")
+					(reference "C51")
 					(unit 1)
 				)
@@
 		(on_board yes)
 		(dnp no)
-		(property "Reference" "C47"
+		(property "Reference" "C49"
 			(at 141.224 127 90)
 			(effects
@@
 			(project "brineomatic"
 				(path "/96477ae2-ef08-48f3-8dd4-fe4478541f68/0f01c39f-0c25-414e-9ed3-1ba09e2af0c5"
-					(reference "C47")
+					(reference "C49")
 					(unit 1)
 				)
@@
 		(on_board yes)
 		(dnp no)
-		(property "Reference" "C51"
+		(property "Reference" "C53"
 			(at 163.83 46.99 0)
 			(effects
@@
 			(project ""
 				(path "/96477ae2-ef08-48f3-8dd4-fe4478541f68/0f01c39f-0c25-414e-9ed3-1ba09e2af0c5"
-					(reference "C51")
+					(reference "C53")
 					(unit 1)
 				)
@@
 		(on_board yes)
 		(dnp no)
-		(property "Reference" "C40"
+		(property "Reference" "C42"
 			(at 100.838 45.72 0)
 			(effects
@@
 			(project "brineomatic"
 				(path "/96477ae2-ef08-48f3-8dd4-fe4478541f68/0f01c39f-0c25-414e-9ed3-1ba09e2af0c5"
-					(reference "C40")
+					(reference "C42")
 					(unit 1)
 				)
@@
 		(on_board yes)
 		(dnp no)
-		(property "Reference" "C46"
+		(property "Reference" "C48"
 			(at 141.224 96.52 90)
 			(effects
@@
 			(project "brineomatic"
 				(path "/96477ae2-ef08-48f3-8dd4-fe4478541f68/0f01c39f-0c25-414e-9ed3-1ba09e2af0c5"
-					(reference "C46")
+					(reference "C48")
 					(unit 1)
 				)
@@
 		(on_board yes)
 		(dnp no)
-		(property "Reference" "C50"
+		(property "Reference" "C52"
 			(at 151.384 127 90)
 			(effects
@@
 			(project "brineomatic"
 				(path "/96477ae2-ef08-48f3-8dd4-fe4478541f68/0f01c39f-0c25-414e-9ed3-1ba09e2af0c5"
-					(reference "C50")
+					(reference "C52")
 					(unit 1)
 				)
@@
 		(on_board yes)
 		(dnp no)
-		(property "Reference" "C38"
+		(property "Reference" "C40"
 			(at 66.04 63.754 0)
 			(effects
@@
 			(project "brineomatic"
 				(path "/96477ae2-ef08-48f3-8dd4-fe4478541f68/0f01c39f-0c25-414e-9ed3-1ba09e2af0c5"
-					(reference "C38")
+					(reference "C40")
 					(unit 1)
 				)
@@
 		(on_board yes)
 		(dnp no)
-		(property "Reference" "C42"
+		(property "Reference" "C44"
 			(at 104.14 92.964 90)
 			(effects
@@
 			(project "brineomatic"
 				(path "/96477ae2-ef08-48f3-8dd4-fe4478541f68/0f01c39f-0c25-414e-9ed3-1ba09e2af0c5"
-					(reference "C42")
+					(reference "C44")
 					(unit 1)
 				)
@@
 		(on_board yes)
 		(dnp no)
-		(property "Reference" "C41"
+		(property "Reference" "C43"
 			(at 104.14 81.28 90)
 			(effects
@@
 			(project "brineomatic"
 				(path "/96477ae2-ef08-48f3-8dd4-fe4478541f68/0f01c39f-0c25-414e-9ed3-1ba09e2af0c5"
-					(reference "C41")
+					(reference "C43")
 					(unit 1)
 				)
@@
 		(on_board yes)
 		(dnp no)
-		(property "Reference" "C45"
+		(property "Reference" "C47"
 			(at 130.556 45.974 0)
 			(effects
@@
 			(project "brineomatic"
 				(path "/96477ae2-ef08-48f3-8dd4-fe4478541f68/0f01c39f-0c25-414e-9ed3-1ba09e2af0c5"
-					(reference "C45")
-					(unit 1)
-				)
+					(reference "C47")
+					(unit 1)
+				)
